File: pcbs/src/mcu_adapter/mcu_adapter.kicad_pcb (KiCad board)
At the start: 2 copper layers, 30 x 21 mm, 3 parts, among them U1 XIAO-THRUHOLE

Commit message: added gerbers
Other:
- outline, holes or cut-outs redrawn
